File: MotorDriver.kicad_sch (KiCad schematic)
At the start: 20 parts, among them J1 Conn_01x04_Pin, J2 Conn_01x02_Pin, J3 Conn_01x02_Pin, J4 Conn_01x03_Pin, U1 L298N, U2 KA78M05_TO252

Commit message: Replaced with new files
Parts:
- removed D9: LED, LED_SMD:LED_0201_0603Metric_Pad0.64x0.40mm_HandSolder, symbol Device:LED
- removed J1: Conn_01x04_Pin, Connector_PinHeader_2.54mm:PinHeader_1x04_P2.54mm_Vertical, symbol Connector:Conn_01x04_Pin
- removed J4: Conn_01x03_Pin, TerminalBlock:TerminalBlock_MaiXu_MX126-5.0-03P_1x03_P5.00mm, symbol Connector:Conn_01x03_Pin
- removed Motor1, Motor2: Conn_01x02_Pin, TerminalBlock_MetzConnect:TerminalBlock_MetzConnect_Type086_RT03402HBLC_1x02_P3.81mm_Horizontal, symbol Connector:Conn_01x02_Pin
- removed U2: KA78M05_TO252, Package_TO_SOT_SMD:TO-252-2, symbol Regulator_Linear:KA78M05_TO252
- added J1: Conn_01x03_Pin, TerminalBlock_Phoenix:TerminalBlock_Phoenix_MKDS-1,5-3_1x03_P5.00mm_Horizontal, symbol Connector:Conn_01x03_Pin
- added J4: Conn_01x04_Pin, Connector_PinHeader_2.54mm:PinHeader_1x04_P2.54mm_Vertical, symbol Connector:Conn_01x04_Pin
- added J5, J6, J7: Conn_01x02_Pin, Connector_PinHeader_2.54mm:PinHeader_1x02_P2.54mm_Vertical, symbol Connector:Conn_01x02_Pin
- added R2: 0.1, Resistor_SMD:R_0201_0603Metric_Pad0.64x0.40mm_HandSolder, symbol Device:R
- added TP1, TP2: TestPoint, TestPoint:TestPoint_Keystone_5005-5009_Compact, symbol Connector:TestPoint
- added U2: L7805, L7805:TO255P1020X450X2000-3, symbol Regulator_Linear:L7805
- C1: value C_Polarized -> 220u; footprint Capacitor_THT:CP_Radial_D5.0mm_P2.50mm -> Capacitor_THT:CP_Radial_D10.0mm_P2.50mm
- C2: value C_Polarized -> 220u; footprint Capacitor_THT:CP_Radial_D5.0mm_P2.50mm -> Capacitor_THT:CP_Axial_L26.5mm_D20.0mm_P33.00mm_Horizontal
- J2: footprint Connector_PinHeader_2.54mm:PinHeader_1x02_P2.54mm_Vertical -> TerminalBlock_Phoenix:TerminalBlock_Phoenix_MKDS-1,5-2_1x02_P5.00mm_Horizontal
- J3: footprint Connector_PinHeader_1.27mm:PinHeader_1x02_P1.27mm_Vertical -> TerminalBlock_Phoenix:TerminalBlock_Phoenix_MKDS-1,5-2_1x02_P5.00mm_Horizontal
- R1: value R -> 0.1
Connections:
- net +5V: now also C2.1, J1.3 (Pin_3), J5.2 (Pin_2), J6.2 (Pin_2), U2.3 (OUT); no longer C1.1, R1.1
- net EnA: now also J6.1 (Pin_1); no longer J2.1 (Pin_1)
- net EnB: now also J5.1 (Pin_1); no longer J2.2 (Pin_2)
- net GND: now also J1.2 (Pin_2), U2.2 (GND); no longer U1.1 (SENSE_A), U1.15 (SENSE_B)
- net at J3.1 (Pin_1): now also D4.2 (A), D8.1 (K), U1.14 (OUT4)
- net input3: now reaches U1.10 (IN3)
- net input3: now also J4.3 (Pin_3)
- net input4: now reaches U1.12 (IN4)
- net input4: now also J4.4 (Pin_4)
- net at D3.2 (A), D7.1 (K), U1.13 (OUT3): now also J3.2 (Pin_2)
- net at D1.2 (A), D5.1 (K), U1.2 (OUT1): now also J2.2 (Pin_2)
- net at D2.2 (A), D6.1 (K), U1.3 (OUT2): now also J2.1 (Pin_1)
- net input1: now reaches U1.5 (IN1)
- net input1: now also J4.1 (Pin_1)
- net input2: now reaches U1.7 (IN2)
- net input2: now also J4.2 (Pin_2)
- net at R1.2: now also TP1.1
- net VCC renamed +12V
- net +12V: now also J1.1 (Pin_1), J7.1 (Pin_1); no longer C2.1, J3.2 (Pin_2)
- new net: R1.1, U1.1 (SENSE_A)
- new net: R2.1, U1.15 (SENSE_B)
- new net: R2.2, TP2.1
- new net: C1.1, J7.2 (Pin_2), U2.1 (IN)
Other:
- title: (none) -> L298MotorDriver
